File: pcb/avrprog.kicad_pcb (KiCad board)
At the start: 2 copper layers, 25 parts, among them IC1 ATMEGA8A-P, P1 USB_B, P2 CONN_02X05, P3 CONN_01X02, P4 CONN_01X01, P5 CONN_02X04, U1 FT232RL

Commit message: pcb (not finished)
Parts:
- added C7: 100nF, Capacitors_THT:C_Rect_L7_W2_P5, F.Cu at (201.9, 120.7)
- added D6: 1N4148, Diodes_THT:Diode_DO-35_SOD27_Horizontal_RM10, F.Cu at (198.1, 130.8)
- R6: value 10K -> 4.7K
- moved C4 50.9 mm to (166.4, 101.6), turned to 270 degrees
- moved U1 42.1 mm to (160.0, 106.7), turned to 180 degrees
- moved P4 41.2 mm to (201.9, 157.5)
- moved C2 41.0 mm to (153.7, 105.4)
- moved C3 39.9 mm to (149.9, 108.0)
- moved P3 21.9 mm to (223.5, 120.7)
- moved L1 19.4 mm to (134.6, 114.3), turned to 90 degrees
- moved C1 16.6 mm to (128.3, 119.4), turned to 0 degrees
- moved D1 10.2 mm to (154.9, 132.1), turned to 90 degrees
- moved D2 10.2 mm to (161.3, 132.1), turned to 90 degrees
- moved C5 4.02 mm to (205.7, 135.9)
- moved R6 4.02 mm to (205.7, 130.8)
- moved P5 4.02 mm to (186.7, 121.9)
- moved R1 4.02 mm to (156.2, 125.7), turned to 90 degrees
- moved IC1 3.81 mm to (208.3, 120.7)
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
Commit message: pcb (not finished)
Parts:
- added D7: green, LEDs:LED-3MM, F.Cu at (138.4, 127.0)
- added D8: green, LEDs:LED-3MM, F.Cu at (229.9, 105.4)
- added P6: CONN_02X05, Pin_Headers:Pin_Header_Straight_2x05, F.Cu at (188.0, 100.3)
- added R7: 1K, Resistors_THT:Resistor_Horizontal_RM10mm, F.Cu at (153.7, 132.1)
- added R8: 1K, Resistors_THT:Resistor_Horizontal_RM10mm, F.Cu at (221.0, 110.5)
- L1: value L_Core_Ferrite -> ferrite bead
- moved P4 36.8 mm to (228.6, 132.1)
- moved P2 33.0 mm to (229.9, 114.3)
- moved C5 24.1 mm to (205.7, 111.8)
- moved P5 23.9 mm to (176.5, 100.3)
- moved C7 21.9 mm to (205.7, 99.1)
- moved P3 21.9 mm to (227.3, 99.1)
- moved R6 21.9 mm to (201.9, 109.2)
- moved C6 21.7 mm to (221.0, 119.4)
- moved IC1 21.6 mm to (209.6, 99.1)
- moved D6 21.6 mm to (198.1, 109.2)
- moved L1 20.5 mm to (153.7, 121.9), turned to 270 degrees
- moved P1 20.5 mm to (149.9, 106.7)
- moved R5 19.4 mm to (193.0, 130.8)
- moved C1 19.2 mm to (147.3, 116.8), turned to 180 degrees
- moved D5 19.1 mm to (185.4, 130.8)
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Connections:
- C1 pad 1: GND -> Net-(C1-Pad1)
- C1 pad 2: Net-(C1-Pad2) -> GND
- L1 pad 1: Net-(C1-Pad2) -> Net-(C1-Pad1)
- P1 pad 1: Net-(C1-Pad2) -> Net-(C1-Pad1)
Routing:
- net GND: track 0.00 -> 189.1 mm, vias 0 -> 5
- net +5V: track 0.00 -> 122.2 mm, vias 0 -> 1
- net RESET: track 0.00 -> 42.2 mm, vias 0 -> 2
- net MOSI: track 0.00 -> 30.6 mm, vias 0 -> 2
- net SCK: track 0.00 -> 29.5 mm, vias 0 -> 2
- net Net-(P2-Pad2): track 0.00 -> 27.7 mm
- net MISO: track 0.00 -> 26.7 mm, vias 0 -> 2
- net Net-(IC1-Pad13): track 0.00 -> 23.7 mm
- net SS: track 0.00 -> 20.6 mm, vias 0 -> 2
- net Net-(IC1-Pad6): track 0.00 -> 20.3 mm, vias 0 -> 2
- net Net-(C4-Pad1): track 0.00 -> 18.9 mm
- net Net-(C1-Pad1): track 0.00 -> 17.7 mm
- net USBDM: track 0.00 -> 17.5 mm, vias 0 -> 2
- net USBDP: track 0.00 -> 11.9 mm
- net Net-(D8-Pad2): track 0.00 -> 8.45 mm
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Other:
- board outline added: 100.3 x 40.6 mm
- net class Default: clearance 0.2 -> 0.15; trace_width 0.25 -> 0.5; via_dia 0.6 -> 1; via_drill 0.4 -> 0.6
- rule trace_clearance: 0.2 -> 0.15
