File: pcb/avrprog.sch (KiCad schematic (older format))
At the start: 25 parts, among them IC1 ATMEGA8A-P, P1 USB_B, P2 CONN_02X05, P3 CONN_01X02, P4 CONN_01X01, P5 CONN_02X04, U1 FT232RL

Commit message: pcb (not finished)
Parts:
- added C7: 100nF, Capacitors_THT:C_Rect_L7_W2_P5, symbol C
- added D6: 1N4148, Diodes_THT:Diode_DO-35_SOD27_Horizontal_RM10, symbol D
- R6: value 10K -> 4.7K
Connections:
- net +5V: now also D6.1 (K)
- net GND: now also C7.2
- net RESET: now also C7.1, D6.2 (A)
Other:
- moved on the sheet: R6
Changed lines of the file:
@@
 L R R6
 U 1 1 5CBDCCE3
-P 6950 1500
-F 0 "R6" V 7030 1500 50  0000 C CNN
-F 1 "10K" V 6950 1500 50  0000 C CNN
-F 2 "Resistors_THT:Resistor_Horizontal_RM10mm" V 6880 1500 50  0001 C CNN
-F 3 "" H 6950 1500 50  0000 C CNN
-	1    6950 1500
+P 6950 1700
+F 0 "R6" V 7030 1700 50  0000 C CNN
+F 1 "4.7K" V 6950 1700 50  0000 C CNN
+F 2 "Resistors_THT:Resistor_Horizontal_RM10mm" V 6880 1700 50  0001 C CNN
+F 3 "" H 6950 1700 50  0000 C CNN
+	1    6950 1700
 	1    0    0    -1
 $EndComp
@@
 	0    1    1    0
 $EndComp
-Wire Wire Line
-	6950 1650 6950 1850
 $Comp
 L +5V #PWR04
@@
 L +5V #PWR05
 U 1 1 5CBE10A7
-P 6950 1350
-F 0 "#PWR05" H 6950 1200 50  0001 C CNN
-F 1 "+5V" H 6950 1490 50  0000 C CNN
-F 2 "" H 6950 1350 50  0000 C CNN
-F 3 "" H 6950 1350 50  0000 C CNN
-	1    6950 1350
+P 6950 1550
+F 0 "#PWR05" H 6950 1400 50  0001 C CNN
+F 1 "+5V" H 6950 1690 50  0000 C CNN
+F 2 "" H 6950 1550 50  0000 C CNN
+F 3 "" H 6950 1550 50  0000 C CNN
+	1    6950 1550
 	1    0    0    -1
 $EndComp
@@
 Text GLabel 8850 2250 2    50   BiDi ~ 0
 MISO
-Text GLabel 6950 1850 0    50   Input ~ 0
+Text GLabel 6350 1850 0    50   Input ~ 0
 RESET
 Text GLabel 3650 4450 2    50   Output ~ 0
@@
 Connection ~ 1850 2600
 Connection ~ 1850 2900
+$Comp
+L C C7
+U 1 1 5CC60C6E
+P 6500 2000
+F 0 "C7" H 6525 2100 50  0000 L CNN
+F 1 "100nF" H 6525 1900 50  0000 L CNN
+F 2 "Capacitors_THT:C_Rect_L7_W2_P5" H 6538 1850 50  0001 C CNN
+F 3 "" H 6500 2000 50  0000 C CNN
+	1    6500 2000
+	1    0    0    -1
+$EndComp
+Wire Wire Line
+	6350 1850 6950 1850
+Connection ~ 6500 1850
+$Comp
+L GND #PWR030
+U 1 1 5CC61DDB
+P 6500 2150
+F 0 "#PWR030" H 6500 1900 50  0001 C CNN
+F 1 "GND" H 6500 2000 50  0000 C CNN
+F 2 "" H 6500 2150 50  0000 C CNN
+F 3 "" H 6500 2150 50  0000 C CNN
+	1    6500 2150
+	1    0    0    -1
+$EndComp
+$Comp
+L D D6
+U 1 1 5CC61E3D
+P 6750 1700
+F 0 "D6" H 6750 1800 50  0000 C CNN
+F 1 "1N4148" H 6750 1600 50  0000 C CNN
+F 2 "Diodes_THT:Diode_DO-35_SOD27_Horizontal_RM10" H 6750 1700 50  0001 C CNN
+F 3 "" H 6750 1700 50  0000 C CNN
+	1    6750 1700
+	0    1    1    0
+$EndComp
+Wire Wire Line
+	6750 1550 6950 1550
+Connection ~ 6750 1850
 $EndSCHEMATC

Commit message: pcb (not finished)
Parts:
- added D7, D8: green, LEDs:LED-3MM, symbol LED
- added P6: CONN_02X05, Pin_Headers:Pin_Header_Straight_2x05, symbol CONN_02X05
- added R7, R8: 1K, Resistors_THT:Resistor_Horizontal_RM10mm, symbol R
- L1: value L_Core_Ferrite -> ferrite bead
Connections:
- net +5V: now also P6.2 (P2), R7.1
- net GND: now also C1.2, D7.1 (K), D8.1 (K), P6.10 (P10), P6.3 (P3), P6.4 (P4), P6.6 (P6), P6.8 (P8); no longer C1.1
- net MISO: now also P6.9 (P9)
- net MOSI: now also P6.1 (P1)
- net RESET: now also P6.5 (P5)
- net SCK: now also P6.7 (P7)
- net at P2.2 (P2), P3.2 (P2): now also R8.1
- net at L1.1, P1.1 (VBUS): now also C1.1; no longer C1.2
- new net: D7.2 (A), R7.2
- new net: D8.2 (A), R8.2
